File: FlybackV2.kicad_sch (KiCad schematic)
At the start: 147 parts, among them J1 Power, J10 ads1256, J11 Coils, J2 Conn_01x02, J3 Conn_01x03, T2 0399-T208, U1 LT8304, U10 LT1634BIS8-2.5, U11 MAX4239, U2 TEA 1-0505, U4 7.68MHz, U5 MAX4239, U6 MAX4239, U7 MAX4239, U8 ADS1256IDBR, U9 MAX4239

Commit message: v2 now with pnp transistor
Parts:
- removed C36: 100nF, Capacitor_SMD:C_0805_2012Metric, symbol Device:C_Small
- removed R58: 1K, Resistor_SMD:R_1206_3216Metric, symbol Device:R_US
- removed R70: 0, Resistor_THT:R_Axial_DIN0309_L9.0mm_D3.2mm_P20.32mm_Horizontal, symbol Device:R_US
- removed R71, R72: 0, Resistor_SMD:R_1206_3216Metric, symbol Device:R_US
- removed U2: TEA 1-0505, JuanDavid_Library:SIP-4_L11.7-W6.0-P2.54_B0505S-1W, symbol JuanDavid_Library:TEA1-0505
- added Q6: 2N3906, Package_TO_SOT_THT:TO-92_Inline, symbol Transistor_BJT:2N3906
- added R12: 560, Resistor_SMD:R_1206_3216Metric, symbol Device:R_US
- added R21: 1K, Resistor_SMD:R_1206_3216Metric, symbol Device:R_US
Connections:
- net 5_{iso}V is gone; now on net +5V: C34.1, C35.1, C4.1, R62.1, R68.1, U11.5 (~{SHDN}), U11.6 (VCC), U3.3 (VIN), U8.1 (AVDD)
- net ADC3 is gone; now on net ADC1: C24.1, R34.2
- net GND2 is gone; now on net GND: C13.2, C16.2, C17.2, C18.2, C19.1, C20.1, C21.2, C22.2, C23.2, C24.2, C25.2, C26.1, C28.1, C29.2, C3.2, C30.2, C31.2, C32.2, C33.2, C34.2, C35.2, C37.2, C39.1, C4.2, C40.2, C5.2, D12.1 (K), D14.2 (A), D23.1, D24.2 (A), D25.2 (A), D26.1 (K), D9.2 (A), J10.6 (Pin_6), R20.1, R20.2, R26.1, R35.2, R38.2, R43.2, R44.2, R46.3, R61.1, T2.7, U10.4, U11.2 (GND), U3.1 (GND), U5.2 (GND), U6.2 (GND), U7.2 (GND), U8.17 (DGND), U8.2 (AGND), U8.5 (AINCOM), U9.2 (GND)
- net +5V: now also Q6.3 (C), R21.1
- net ADC0: now also U7.1 (OUT), U7.4 (IN-)
- net ADC1: no longer U9.1 (OUT), U9.4 (IN-)
- net ADC2: now also U9.1 (OUT), U9.4 (IN-); no longer U7.1 (OUT), U7.4 (IN-)
- net at R1.2, R11.1, R2.2: now also Q6.1 (E); no longer Q1.3
- new net: Q6.2 (B), R12.1, R21.2
- new net: Q1.3, R12.2
- no-connect marks 9 -> 10
Other:
- moved on the sheet: C1, C10, C12, C13, C14, C15, C17, C2, C3, C4, C5, C7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

Commit message: finish v2 version
Parts:
- removed R20: 0, Resistor_THT:R_Axial_DIN0309_L9.0mm_D3.2mm_P25.40mm_Horizontal, symbol Device:R_US
- removed R27: 0, Resistor_THT:R_Axial_DIN0309_L9.0mm_D3.2mm_P20.32mm_Horizontal, symbol Device:R_US
- removed R30: 100, Resistor_THT:R_Axial_DIN0207_L6.3mm_D2.5mm_P10.16mm_Horizontal, symbol Device:R_US
- added C36, C41, C42: 10u, Capacitor_SMD:C_0805_2012Metric, symbol Device:C_Polarized_US
- added R58: 100, Resistor_SMD:R_1206_3216Metric, symbol Device:R_US
- D12: footprint Resistor_THT:R_Axial_DIN0411_L9.9mm_D3.6mm_P7.62mm_Vertical -> LED_SMD:LED_0805_2012Metric
- R26: value 47M -> 100K
Connections:
- net +3.3_{iso}V: now also C36.1, C42.1
- net +5V: now also Q6.1 (E), C41.1; no longer Q6.3 (C)
- net GND: now also C36.2, C41.2, C42.2
- net In_{pos}: now also R58.1
- net at C39.2, D25.1 (K), U5.3 (IN+): now also R58.2
- net at R1.2, R11.1, R2.2: now also Q6.3 (C); no longer Q6.1 (E)

Commit message: init: new version
Parts:
- removed C18, C31, C32: 100nF, Capacitor_SMD:C_0805_2012Metric, symbol Device:C_Small
- removed C21, C22, C23, C24, C30, C36, C41: 10u, Capacitor_SMD:C_0805_2012Metric, symbol Device:C_Polarized_US
- removed C25, C28: 20pF, Capacitor_SMD:C_0805_2012Metric, symbol Device:C_Small
- removed C26, C27, C38, C39: 1u, Capacitor_SMD:C_0805_2012Metric, symbol Device:C_Small
- removed C29, C34, C37: 10u, Capacitor_SMD:C_0805_2012Metric, symbol Device:C_Small
- removed C33, C35, C40: 0.1u, Capacitor_SMD:C_0805_2012Metric, symbol Device:C_Small
- removed D19, D21: D_Small_Filled, Diode_THT:D_A-405_P10.16mm_Horizontal, symbol Device:D_Small_Filled
- removed D20, D22: LED, LED_SMD:LED_0805_2012Metric, symbol Device:LED
- removed D23: SMBJ5.0CA, JuanDavid_Library:SMB_L4.6-W3.6-LS5.3-BI, symbol JuanDavid_Library:SMBJ5.0CA
- removed D24, D25: D_Zener_Small_Filled, Diode_THT:D_A-405_P10.16mm_Horizontal, symbol Device:D_Zener_Small_Filled
- removed J10: ads1256, Connector_PinHeader_2.54mm:PinHeader_1x06_P2.54mm_Vertical, symbol Connector_Generic:Conn_01x06
- removed J11: Coils, Connector_PinHeader_2.54mm:PinHeader_1x06_P2.54mm_Vertical, symbol Connector_Generic:Conn_01x06
- removed Q2, Q3: ~, JuanDavid_Library:TO-92-3_L4.9-W3.7-P2.54-L, symbol JuanDavid_Library:2N3904
- removed R17, R18, R43, R44, R51, R52, R57, R65: 1K, Resistor_SMD:R_1206_3216Metric, symbol Device:R_US
- removed R23, R24, R25, R28, R29, R31, R34, R55, R56, R58, R59: 100, Resistor_SMD:R_1206_3216Metric, symbol Device:R_US
- removed R35: 10K, Resistor_SMD:R_1206_3216Metric, symbol Device:R_US
- removed R36, R39: 2.2K, Resistor_SMD:R_1206_3216Metric, symbol Device:R_US
- removed R37, R40: 6.8K, Resistor_SMD:R_1206_3216Metric, symbol Device:R_US
- removed R38: 10, Resistor_SMD:R_1206_3216Metric, symbol Device:R_US
- removed R45, R46: ~, JuanDavid_Library:RELAY-TH_SRD-XXVDC-XL-C, symbol JuanDavid_Library:SimpleRelay
- removed R47, R48: 560, Resistor_SMD:R_1206_3216Metric, symbol Device:R_US
- removed R61, R68: 0, Resistor_SMD:R_1206_3216Metric, symbol Device:R_US
- removed R62: 4, Resistor_SMD:R_1206_3216Metric, symbol Device:R_US
- removed U10: LT1634BIS8-2.5, JuanDavid_Library:SO-8_L4.9-W3.9-P1.27-LS5.9-BL, symbol JuanDavid_Library:LT1634BIS8-2.5
- removed U11, U5, U6, U7: MAX4239, JuanDavid_Library:SOT-23-6_L2.9-W1.6-P0.95-LS2.9-BL, symbol JuanDavid_Library:MAX4239
- removed U4: 7.68MHz, JuanDavid_Library:CRYSTAL-SMD_L11.4-W4.7-LS12.4, symbol JuanDavid_Library:7.68MHz
- removed U8: ADS1256IDBR, JuanDavid_Library:SSOP-28_L10.2-W5.3-P0.65-LS7.8-BL, symbol JuanDavid_Library:ADS1256IDBR
- added J4: Coils, symbol Connector_Generic:Conn_01x05
- J2: value Conn_01x02 -> Divisor; footprint Connector_PinHeader_2.54mm:PinHeader_1x02_P2.54mm_Vertical -> (none)
- R67: value 1K -> 2M; footprint Resistor_SMD:R_1206_3216Metric -> Resistor_THT:R_Axial_DIN0207_L6.3mm_D2.5mm_P15.24mm_Horizontal
Connections:
- net In_{pos} is gone; now on an unnamed net: J2.1 (Pin_1)
- net +5V: now also J4.1 (Pin_1); no longer R67.2
- net 500V: now also R67.2; no longer R32.3
- net GND: now also J2.2 (Pin_2), J4.5 (Pin_5)
- net GPIO_{EN}: now also J4.2 (Pin_2)
- net GPIO_{K1}: now also J4.4 (Pin_4)
- net GPIO_{K2}: now also J4.3 (Pin_3)
- net at R67.1: now also R32.3
- net at R41.1, R42.1: now also J3.1 (Pin_1)
- net ADC2: no longer names the net of U9.1 (OUT), U9.4 (IN-)
- no-connect marks 10 -> 1
Other:
- moved on the sheet: C16, C19, C20, C42, D14, D15, D16, D17, D18, D6, D7, D9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
